File: fourscore.kicad_sch (KiCad schematic)
At the start: 33 parts, among them J1 Conn_01x07_Socket, J2 Conn_01x07_Socket, J3 Conn_01x07_Socket, J4 Conn_01x07_Socket, J5 Conn_01x07_Socket, SW1 2-4, SW2 B, SW3 A

Commit message: dealt with all warnings
Parts:
- C2: footprint Capacitor_THT:C_Axial_L3.8mm_D2.6mm_P7.50mm_Horizontal -> Capacitor_THT:C_Rect_L9.0mm_W2.5mm_P7.50mm_MKT
Changed lines of the file:
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@@
 	(paper "A4")
 	(junction
+		(at 49.53 133.35)
+		(diameter 0)
+		(color 0 0 0 0)
+	)
+	(junction
 		(at 137.16 78.74)
 		(diameter 0)
@@
 	)
 	(junction
+		(at 62.23 133.35)
+		(diameter 0)
+		(color 0 0 0 0)
+	)
+	(junction
 		(at -128.27 62.23)
 		(diameter 0)
@@
 	(wire
 		(pts
+			(xy 62.23 133.35) (xy 59.69 133.35)
+		)
+		(stroke
+			(width 0)
+			(type default)
+		)
+	)
+	(wire
+		(pts
 			(xy 160.02 163.83) (xy 163.83 163.83)
 		)
@@
 	(wire
 		(pts
+			(xy 49.53 133.35) (xy 52.07 133.35)
+		)
+		(stroke
+			(width 0)
+			(type default)
+		)
+	)
+	(wire
+		(pts
 			(xy 106.68 78.74) (xy 109.22 78.74)
 		)
@@
 	(symbol
 		(lib_id "power:GND")
-		(at 52.07 133.35 270)
+		(at 49.53 133.35 270)
 		(unit 1)
 		(exclude_from_sim no)
@@
 		(fields_autoplaced yes)
 		(property "Reference" "#PWR07"
-			(at 45.72 133.35 0)
+			(at 43.18 133.35 0)
 			(effects
 				(font
@@
 		)
 		(property "Value" "GND"
-			(at 48.26 133.3499 90)
+			(at 45.72 133.3499 90)
 			(effects
 				(font
@@
 		)
 		(property "Footprint" ""
-			(at 52.07 133.35 0)
+			(at 49.53 133.35 0)
 			(effects
 				(font
@@
 		)
 		(property "Datasheet" ""
-			(at 52.07 133.35 0)
+			(at 49.53 133.35 0)
 			(effects
 				(font
@@
 		)
 		(property "Description" "Power symbol creates a global label with name \"GND\" , ground"
-			(at 52.07 133.35 0)
+			(at 49.53 133.35 0)
 			(effects
 				(font
@@
 	)
 	(symbol
+		(lib_id "power:PWR_FLAG")
+		(at 49.53 133.35 0)
+		(unit 1)
+		(exclude_from_sim no)
+		(in_bom yes)
+		(on_board yes)
+		(dnp no)
+		(fields_autoplaced yes)
+		(property "Reference" "#FLG01"
+			(at 49.53 131.445 0)
+			(effects
+				(font
+					(size 1.27 1.27)
+				)
+				(hide yes)
+			)
+		)
+		(property "Value" "PWR_FLAG"
+			(at 49.53 128.27 0)
+			(effects
+				(font
+					(size 1.27 1.27)
+				)
+			)
+		)
+		(property "Footprint" ""
+			(at 49.53 133.35 0)
+			(effects
+				(font
+					(size 1.27 1.27)
+				)
+				(hide yes)
+			)
+		)
+		(property "Datasheet" "~"
+			(at 49.53 133.35 0)
+			(effects
+				(font
+					(size 1.27 1.27)
+				)
+				(hide yes)
+			)
+		)
+		(property "Description" "Special symbol for telling ERC where power comes from"
+			(at 49.53 133.35 0)
+			(effects
+				(font
+					(size 1.27 1.27)
+				)
+				(hide yes)
+			)
+		)
+		(pin "1"
+		)
+		(instances
+			(project "fourscore"
+				(path "/31768e27-9928-4290-91bf-3a747329480b"
+					(reference "#FLG01")
+					(unit 1)
+				)
+			)
+		)
+	)
+	(symbol
 		(lib_id "power:GND")
 		(at 139.7 152.4 270)
@@
 	)
 	(symbol
+		(lib_id "power:PWR_FLAG")
+		(at 62.23 133.35 0)
+		(unit 1)
+		(exclude_from_sim no)
+		(in_bom yes)
+		(on_board yes)
+		(dnp no)
+		(fields_autoplaced yes)
+		(property "Reference" "#FLG02"
+			(at 62.23 131.445 0)
+			(effects
+				(font
+					(size 1.27 1.27)
+				)
+				(hide yes)
+			)
+		)
+		(property "Value" "PWR_FLAG"
+			(at 62.23 128.27 0)
+			(effects
+				(font
+					(size 1.27 1.27)
+				)
+			)
+		)
+		(property "Footprint" ""
+			(at 62.23 133.35 0)
+			(effects
+				(font
+					(size 1.27 1.27)
+				)
+				(hide yes)
+			)
+		)
+		(property "Datasheet" "~"
+			(at 62.23 133.35 0)
+			(effects
+				(font
+					(size 1.27 1.27)
+				)
+				(hide yes)
+			)
+		)
+		(property "Description" "Special symbol for telling ERC where power comes from"
+			(at 62.23 133.35 0)
+			(effects
+				(font
+					(size 1.27 1.27)
+				)
+				(hide yes)
+			)
+		)
+		(pin "1"
+		)
+		(instances
+			(project "fourscore"
+				(path "/31768e27-9928-4290-91bf-3a747329480b"
+					(reference "#FLG02")
+					(unit 1)
+				)
+			)
+		)
+	)
+	(symbol
 		(lib_id "Connector:Conn_01x07_Socket")
 		(at 114.3 67.31 90)
@@
 			)
 		)
-		(property "Footprint" "Capacitor_THT:C_Axial_L3.8mm_D2.6mm_P7.50mm_Horizontal"
+		(property "Footprint" "Capacitor_THT:C_Rect_L9.0mm_W2.5mm_P7.50mm_MKT"
 			(at 164.7952 171.45 0)
 			(effects
@@
 	(symbol
 		(lib_id "power:VCC")
-		(at 59.69 133.35 270)
+		(at 62.23 133.35 270)
 		(unit 1)
 		(exclude_from_sim no)
@@
 		(fields_autoplaced yes)
 		(property "Reference" "#PWR017"
-			(at 55.88 133.35 0)
+			(at 58.42 133.35 0)
 			(effects
 				(font
@@
 		)
 		(property "Value" "VCC"
-			(at 63.5 133.3499 90)
+			(at 66.04 133.3499 90)
 			(effects
 				(font
@@
 		)
 		(property "Footprint" ""
-			(at 59.69 133.35 0)
+			(at 62.23 133.35 0)
 			(effects
 				(font
@@
 		)
 		(property "Datasheet" ""
-			(at 59.69 133.35 0)
+			(at 62.23 133.35 0)
 			(effects
 				(font
@@
 		)
 		(property "Description" "Power symbol creates a global label with name \"VCC\""
-			(at 59.69 133.35 0)
+			(at 62.23 133.35 0)
 			(effects
 				(font
